Commit message: 주행시야 갱신

File: urdf/turtlebot3_waffle_gamma.gazebo.xacro (robot description, xacro)
@@ -12,5 +12,5 @@
     <kp>500000.0</kp>
     <kd>10.0</kd>
-    <minDepth>0.001</minDepth>
+    <minDepth>0.0</minDepth> # 0.001
     <maxVel>1.0</maxVel> # 0.1
     <fdir1>1 0 0</fdir1>
@@ -22,5 +22,5 @@
     <kp>500000.0</kp>
     <kd>10.0</kd>
-    <minDepth>0.001</minDepth>
+    <minDepth>0.0</minDepth> # 0.001
     <maxVel>1.0</maxVel> # 0.1
     <fdir1>1 0 0</fdir1>
@@ -32,5 +32,5 @@
     <kp>1000000.0</kp>
     <kd>100.0</kd>
-    <minDepth>0.001</minDepth>
+    <minDepth>0.0</minDepth> # 0.001
     <maxVel>1.0</maxVel>
     <material>Gazebo/FlatBlack</material>
@@ -41,5 +41,5 @@
     <kp>1000000.0</kp>
     <kd>100.0</kd>
-    <minDepth>0.001</minDepth>
+    <minDepth>0.0</minDepth> # 0.001
     <maxVel>1.0</maxVel>
     <material>Gazebo/FlatBlack</material>

File: urdf/turtlebot3_waffle_gamma.urdf.xacro (robot description, xacro)
@@ -31,5 +31,6 @@
     <inertial>
       <origin xyz="0 0 0" rpy="0 0 0"/>
-      <mass value="1.3729096e+00"/>
+      <!-- <mass value="1.3729096e+00"/> -->
+      <mass value="0.1"/>
       <inertia ixx="8.7002718e-03" ixy="-4.7576583e-05" ixz="1.1160499e-04"
                iyy="8.6195418e-03" iyz="-3.5422299e-06"
@@ -59,5 +60,6 @@
     <inertial>
       <origin xyz="0 0 0" />
-      <mass value="2.8498940e-02" />
+      <!-- <mass value="2.8498940e-02" /> -->
+      <mass value="0.1"/>
       <inertia ixx="1.1175580e-05" ixy="-4.2369783e-11" ixz="-5.9381719e-09"
                iyy="1.1192413e-05" iyz="-1.4400107e-11"
@@ -87,5 +89,6 @@
     <inertial>
       <origin xyz="0 0 0" />
-      <mass value="2.8498940e-02" />
+      <!-- <mass value="2.8498940e-02" /> -->
+      <mass value="0.1"/>
       <inertia ixx="1.1175580e-05" ixy="-4.2369783e-11" ixz="-5.9381719e-09"
                iyy="1.1192413e-05" iyz="-1.4400107e-11"
@@ -173,5 +176,6 @@
   <joint name="camera_joint" type="fixed">
     <!-- <origin xyz="0.064 -0.065 0.094" rpy="0 0 0"/> -->
-    <origin xyz="0.128 -0.065 0.094" rpy="0 0 0"/>
+    <!-- <origin xyz="0.128 -0.065 0.094" rpy="0 0 0"/> -->
+    <origin xyz="0.128 -0.065 0.5" rpy="0 0 0"/>
     <parent link="base_link"/>
     <child link="camera_link"/>
