Commit message: 실제로봇 적용

File: urdf/turtlebot3_waffle_beta.urdf.xacro (robot description, xacro)
@@ -2,5 +2,4 @@
 <robot name="turtlebot3_waffle" xmlns:xacro="http://ros.org/wiki/xacro">
   <xacro:include filename="$(find turtlebot3_description)/urdf/common_properties.xacro"/>
-  <xacro:include filename="$(find turtlebot3_description)/urdf/turtlebot3_waffle.gazebo.xacro"/>
   <xacro:property name="r200_cam_rgb_px" value="0.005"/>
   <xacro:property name="r200_cam_rgb_py" value="0.018"/>

File: urdf/turtlebot3_waffle_gamma.urdf.xacro (robot description, xacro)
@@ -2,5 +2,4 @@
 <robot name="turtlebot3_waffle" xmlns:xacro="http://ros.org/wiki/xacro">
   <xacro:include filename="$(find turtlebot3_description)/urdf/common_properties.xacro"/>
-  <xacro:include filename="$(find shared_control)/urdf/turtlebot3_waffle_gamma.gazebo.xacro"/>
   <xacro:property name="r200_cam_rgb_px" value="0.005"/>
   <xacro:property name="r200_cam_rgb_py" value="0.018"/>
@@ -149,5 +148,5 @@
     <child link="base_scan"/>
     <!-- <origin xyz="-0.064 0 0.122" rpy="0 0 0"/> -->
-    <origin xyz="0 0 0.130" rpy="0 0 1.539"/>
+    <origin xyz="0 0 0.130" rpy="0 0 -1.539"/>
   </joint>
   <link name="base_scan">
@@ -177,5 +176,5 @@
     <!-- <origin xyz="0.064 -0.065 0.094" rpy="0 0 0"/> -->
     <!-- <origin xyz="0.128 -0.065 0.094" rpy="0 0 0"/> -->
-    <origin xyz="0.128 -0.065 0.5" rpy="0 0 0"/>
+    <origin xyz="0.128 -0.065 0.094" rpy="0 -0.5 0"/>
     <parent link="base_link"/>
     <child link="camera_link"/>

File: urdf/turtlebot3_waffle_gazebo.urdf.xacro (robot description, xacro)
@@ -2,4 +2,5 @@
 <robot name="turtlebot3_waffle" xmlns:xacro="http://ros.org/wiki/xacro">
   <xacro:include filename="$(find turtlebot3_description)/urdf/common_properties.xacro"/>
+  <xacro:include filename="$(find shared_control)/urdf/turtlebot3_waffle_gamma.gazebo.xacro"/>
   <xacro:property name="r200_cam_rgb_px" value="0.005"/>
   <xacro:property name="r200_cam_rgb_py" value="0.018"/>
@@ -14,5 +15,6 @@
   <link name="base_link">
     <visual>
-      <origin xyz="-0.064 0 0.0" rpy="0 0 0"/>
+      <!-- <origin xyz="-0.064 0 0.0" rpy="0 0 0"/> -->
+      <origin xyz="0 0 0" rpy="0 0 0"/>
       <geometry>
         <mesh filename="package://turtlebot3_description/meshes/bases/waffle_base.stl" scale="0.001 0.001 0.001"/>
@@ -21,5 +23,6 @@
     </visual>
     <collision>
-      <origin xyz="-0.064 0 0.047" rpy="0 0 0"/>
+      <!-- <origin xyz="-0.064 0 0.047" rpy="0 0 0"/> -->
+      <origin xyz="0 0 0.047" rpy="0 0 0"/>
       <geometry>
         <box size="0.266 0.266 0.094"/>
@@ -28,5 +31,6 @@
     <inertial>
       <origin xyz="0 0 0" rpy="0 0 0"/>
-      <mass value="1.3729096e+00"/>
+      <!-- <mass value="1.3729096e+00"/> -->
+      <mass value="0.1"/>
       <inertia ixx="8.7002718e-03" ixy="-4.7576583e-05" ixz="1.1160499e-04"
                iyy="8.6195418e-03" iyz="-3.5422299e-06"
@@ -56,5 +60,6 @@
     <inertial>
       <origin xyz="0 0 0" />
-      <mass value="2.8498940e-02" />
+      <!-- <mass value="2.8498940e-02" /> -->
+      <mass value="0.1"/>
       <inertia ixx="1.1175580e-05" ixy="-4.2369783e-11" ixz="-5.9381719e-09"
                iyy="1.1192413e-05" iyz="-1.4400107e-11"
@@ -84,5 +89,6 @@
     <inertial>
       <origin xyz="0 0 0" />
-      <mass value="2.8498940e-02" />
+      <!-- <mass value="2.8498940e-02" /> -->
+      <mass value="0.1"/>
       <inertia ixx="1.1175580e-05" ixy="-4.2369783e-11" ixz="-5.9381719e-09"
                iyy="1.1192413e-05" iyz="-1.4400107e-11"
@@ -93,5 +99,6 @@
     <parent link="base_link"/>
     <child link="caster_back_right_link"/>
-    <origin xyz="-0.177 -0.064 -0.004" rpy="-1.57 0 0"/>
+    <!-- <origin xyz="-0.177 -0.064 -0.004" rpy="-1.57 0 0"/> -->
+    <origin xyz="-0.113 -0.016 -0.004" rpy="-1.57 0 0"/>
   </joint>
   <link name="caster_back_right_link">
@@ -113,5 +120,6 @@
     <parent link="base_link"/>
     <child link="caster_back_left_link"/>
-    <origin xyz="-0.177 0.064 -0.004" rpy="-1.57 0 0"/>
+    <!-- <origin xyz="-0.177 0.064 -0.004" rpy="-1.57 0 0"/> -->
+    <origin xyz="-0.113 0.016 -0.004" rpy="-1.57 0 0"/>
   </joint>
   <link name="caster_back_left_link">
@@ -133,5 +141,6 @@
     <parent link="base_link"/>
     <child link="imu_link"/>
-    <origin xyz="0.0 0 0.068" rpy="0 0 0"/>
+    <!-- <origin xyz="0.0 0 0.068" rpy="0 0 0"/> -->
+    <origin xyz="0.028 -0.0215 0.017" rpy="0 0 0"/>
   </joint>
   <link name="imu_link"/>
@@ -139,5 +148,6 @@
     <parent link="base_link"/>
     <child link="base_scan"/>
-    <origin xyz="-0.064 0 0.122" rpy="0 0 0"/>
+    <!-- <origin xyz="-0.064 0 0.122" rpy="0 0 0"/> -->
+    <origin xyz="0 0 0.130" rpy="0 0 1.539"/>
   </joint>
   <link name="base_scan">
@@ -145,5 +155,6 @@
       <origin xyz="0 0 0" rpy="0 0 0"/>
       <geometry>
-        <mesh filename="package://turtlebot3_description/meshes/sensors/lds.stl" scale="0.001 0.001 0.001"/>
+        <mesh filename="package://turtlebot3_description/meshes/sensors/lds.stl"
+              scale="0.001 0.001 0.001"/>
       </geometry>
       <material name="dark"/>
@@ -164,5 +175,7 @@
   </link>
   <joint name="camera_joint" type="fixed">
-    <origin xyz="0.064 -0.065 0.094" rpy="0 0 0"/>
+    <!-- <origin xyz="0.064 -0.065 0.094" rpy="0 0 0"/> -->
+    <!-- <origin xyz="0.128 -0.065 0.094" rpy="0 0 0"/> -->
+    <origin xyz="0.128 -0.065 0.5" rpy="0 0 0"/>
     <parent link="base_link"/>
     <child link="camera_link"/>
@@ -176,17 +189,9 @@
     </visual>
     <collision>
-      <origin xyz="0.003 0.065 0.007" rpy="0 0 0"/>
+      <origin xyz="0.003 0.065 0.011" rpy="0 0 0"/>
       <geometry>
         <box size="0.012 0.132 0.020"/>
       </geometry>
     </collision>
-    <!-- This inertial field needs doesn't contain reliable data!! -->
-<!--   <inertial>
-      <mass value="0.564" />
-      <origin xyz="0 0 0" />
-      <inertia ixx="0.003881243" ixy="0.0" ixz="0.0"
-               iyy="0.000498940" iyz="0.0"
-               izz="0.003879257" />
-    </inertial>-->
   </link>
   <joint name="camera_rgb_joint" type="fixed">
